Commit message: UPLOADING FILES ...

File: Prácticas/Ejemplos/Ejercicio Opcional PyBullet/src/urdf/ejercicio_opcional_pybullet.urdf (robot description, URDF)
Before this commit: robot myrobot, 3 links, 2 joints
Links:
- removed link arm_link
- added link top_link, mass 1.0; collision box size=0.1 0.7 0.2; visual box size=0.1 0.7 0.1
Joints:
- removed joint body_to_arm
- added joint body_to_top: type continuous, parent body_link, child top_link, origin xyz=0.05 0 0.1, axis 0 0 1
