Commit message: UPLOADING FILES ...

File: Prácticas/Práctica 2: Diseño 3D de un Robot en Blender/src/robot_model/urdf/robot_model.urdf (robot description, URDF)
Before this commit: robot robot_model, 16 links, 15 joints
Links:
- link arm_1_link: mass None -> 5.00000; geometry collision mesh filename=../meshes/dae/Cylinder.015.dae scale=0.20000 0.20000 0.10000; visual mesh filename=../meshes/dae/Cylinder.015.dae scale=0.20000 0.20000 0.10000
- link arm_2_link: mass None -> 5.00000; geometry collision mesh filename=../meshes/dae/Cylinder.017.dae scale=0.20000 0.20000 0.10000; visual mesh filename=../meshes/dae/Cylinder.017.dae scale=0.20000 0.20000 0.10000
- link arm_base_link: mass None -> 5.00000; geometry collision cylinder length=0.20000 radius=0.30000; visual cylinder length=0.20000 radius=0.30000
- link arm_column_link: mass None -> 10.00000; geometry collision cylinder length=1.50000 radius=0.15000; visual cylinder length=1.50000 radius=0.15000
- link arm_gripper_link: mass None -> 10.00000; geometry collision mesh filename=../meshes/dae/Cube.007.dae scale=0.35000 0.15000 0.02500; visual mesh filename=../meshes/dae/Cube.007.dae scale=0.35000 0.15000 0.02500
- link chasis_link: mass None -> 100.00000; geometry collision mesh filename=../meshes/dae/Cube.003.dae scale=0.05000 1.00000 0.35000; visual mesh filename=../meshes/dae/Cube.003.dae scale=0.05000 1.00000 0.35000
- link gripper_left_link: mass None -> 5.00000; geometry collision mesh filename=../meshes/dae/Cube.009.dae scale=0.30000 0.15000 0.02500; visual mesh filename=../meshes/dae/Cube.009.dae scale=0.30000 0.15000 0.02500
- link gripper_right_link: mass None -> 5.00000; geometry collision mesh filename=../meshes/dae/Cube.008.dae scale=0.30000 0.15000 0.02500; visual mesh filename=../meshes/dae/Cube.008.dae scale=0.30000 0.15000 0.02500
- link subjection_down_left_wheel_link: mass None -> 10.00000; geometry collision mesh filename=../meshes/dae/Cylinder.009.dae scale=0.05000 0.05000 0.20000; visual mesh filename=../meshes/dae/Cylinder.009.dae scale=0.05000 0.05000 0.20000
- link subjection_down_right_wheel_link: mass None -> 10.00000; geometry collision mesh filename=../meshes/dae/Cylinder.004.dae scale=0.05000 0.05000 0.20000; visual mesh filename=../meshes/dae/Cylinder.004.dae scale=0.05000 0.05000 0.20000
- link subjection_up_left_wheel_link: mass None -> 10.00000; geometry collision mesh filename=../meshes/dae/Cylinder.010.dae scale=0.05000 0.05000 0.20000; visual mesh filename=../meshes/dae/Cylinder.010.dae scale=0.05000 0.05000 0.20000
- link subjection_up_right_wheel_link: mass None -> 10.00000; geometry collision mesh filename=../meshes/dae/Cylinder.011.dae scale=0.05000 0.05000 0.20000; visual mesh filename=../meshes/dae/Cylinder.011.dae scale=0.05000 0.05000 0.20000
- link wheel_down_left_link: mass None -> 10.00000; geometry collision mesh filename=../meshes/dae/Cylinder.002.dae scale=0.05000 0.05000 0.20000; visual mesh filename=../meshes/dae/Cylinder.002.dae scale=0.05000 0.05000 0.20000
- link wheel_down_right_link: mass None -> 10.00000; geometry collision mesh filename=../meshes/dae/Cylinder.003.dae scale=0.05000 0.05000 0.20000; visual mesh filename=../meshes/dae/Cylinder.003.dae scale=0.05000 0.05000 0.20000
- link wheel_up_left_link: mass None -> 10.00000; geometry collision mesh filename=../meshes/dae/Cylinder.001.dae scale=0.05000 0.05000 0.20000; visual mesh filename=../meshes/dae/Cylinder.001.dae scale=0.05000 0.05000 0.20000
- link wheel_up_right_link: mass None -> 10.00000; geometry collision mesh filename=../meshes/dae/Cylinder.dae scale=0.05000 0.05000 0.20000; visual mesh filename=../meshes/dae/Cylinder.dae scale=0.05000 0.05000 0.20000

Commit message: UPLOADING FILES ...

File: Prácticas/Práctica 2: Diseño 3D de un Robot en Blender/src/robot_model/urdf/robot_model.urdf (robot description, URDF)
Before this commit: robot robot_model, 16 links, 15 joints
Links:
- added link box_down_side_link, mass 10.00000; collision box size=0.10000 0.80000 0.70000; visual box size=0.10000 0.80000 0.70000
- added link box_left_side_link, mass 10.00000; collision box size=0.10000 2.00000 0.70000; visual box size=0.10000 2.00000 0.70000
- added link box_right_side_link, mass 10.00000; collision box size=0.10000 2.00000 0.70000; visual box size=0.10000 2.00000 0.70000
- added link box_up_side_link, mass 10.00000; collision box size=0.10000 0.80000 0.70000; visual box size=0.10000 0.80000 0.70000
- link chasis_link: geometry collision box size=1.00000 4.00000 1.00000; visual mesh filename=../meshes/dae/Cube.003.dae scale=0.05000 1.00000 0.35000
Joints:
- added joint box_down_side_link_joint: type fixed, parent chasis_link, child box_down_side_link, origin xyz=0.00000 1.86075 0.77413 rpy=0.00000 0.00000 1.57080
- added joint box_left_side_link_joint: type fixed, parent chasis_link, child box_left_side_link, origin xyz=0.45000 0.91075 0.77413 rpy=0.00000 0.00000 0.00000
- added joint box_right_side_link_joint: type fixed, parent chasis_link, child box_right_side_link, origin xyz=-0.45000 0.91075 0.77413 rpy=0.00000 0.00000 0.00000
- added joint box_up_side_link_joint: type fixed, parent chasis_link, child box_up_side_link, origin xyz=0.00000 -0.03925 0.77413 rpy=0.00000 0.00000 1.57080
