Commit message: UPLOADING FILES ...

File: Prácticas/Práctica 3: Simulación de Robots usando Middleware/src/robot_model_description/urdf/sensors/camera.urdf.xacro (robot description, xacro)
@@ -3,5 +3,5 @@
   <xacro:macro name="camera" params="parent" >
     <joint name="camera_link_joint" type="fixed">
-      <origin rpy="-3.14159 0.00000 -3.14159" xyz="0.00000 -1.90000 0.45000"/>
+      <origin rpy="0.00000 0.00000 -1.57000" xyz="0.00000 -1.90000 0.65000"/>
       <parent link="${parent}"/>
       <child link="camera_link"/>
@@ -9,5 +9,5 @@
     <link name="camera_link">
       <visual name="camera">
-        <origin rpy="3.14159 -1.57080 3.14159" xyz="0.00000 0.00000 0.00000"/>
+        <origin rpy="0.00000 0.00000 0.00000" xyz="0.00000 0.00000 -0.20000"/>
         <material name="black.007"/>
         <geometry>

File: Prácticas/Práctica 3: Simulación de Robots usando Middleware/src/robot_model_description/urdf/sensors/sensors.urdf.xacro (robot description, xacro)
@@ -3,5 +3,5 @@
   <xacro:macro name="sensors"  params="parent">
     <joint name="sensors_link_joint" type="fixed">
-      <origin rpy="-3.14159 0.00000 -3.14159" xyz="0.00000 0.00000 -1.25000"/>
+      <origin rpy="0.00000 1.57000 -1.57000" xyz="0.00000 0.00000 -1.25000"/>
       <parent link="${parent}"/>
       <child link="sensors_link"/>
@@ -9,5 +9,5 @@
     <link name="sensors_link">
       <visual name="sensors">
-        <origin rpy="3.14159 -1.57080 3.14159" xyz="0.00000 0.00000 0.00000"/>
+        <origin rpy="0.00000 0.00000 0.00000" xyz="0.00000 0.00000 0.00000"/>
         <material name="black.007"/>
         <geometry>
