Commit message: UPLOADING FILES ...

File: Prácticas/Práctica 3: Simulación de Robots usando Middleware/src/robot_model_description/robots/robot.urdf.xacro (robot description, xacro)
@@ -2,13 +2,13 @@
 <robot name="robot_model" xmlns:xacro="http://wiki.ros.org/xacro">
     <!-- includes -->
-    <xacro:include filename="$(find robot_description)/urdf/base/robot_base.urdf.xacro"/>
-    <xacro:include filename="$(find robot_description)/urdf/wheels/rover_wheel.urdf.xacro"/>
-    <xacro:include filename="$(find robot_description)/urdf/arm/scara.urdf.xacro"/>
-    <xacro:include filename="$(find robot_description)/urdf/arm/gripper.urdf.xacro"/>
-    <xacro:include filename="$(find robot_description)/urdf/ros2_control.urdf.xacro"/>
-    <xacro:include filename="$(find robot_description)/urdf/utils/utils.urdf.xacro"/>
-    <xacro:include filename="$(find robot_description)/urdf/sensors/camera.urdf.xacro"/>
-    <xacro:include filename="$(find robot_description)/urdf/sensors/imu_sensor.urdf.xacro"/>
-    <xacro:include filename="$(find robot_description)/urdf/sensors/sensors.urdf.xacro"/>
+    <xacro:include filename="$(find robot_model_description)/urdf/base/robot_base.urdf.xacro"/>
+    <xacro:include filename="$(find robot_model_description)/urdf/wheels/rover_wheel.urdf.xacro"/>
+    <xacro:include filename="$(find robot_model_description)/urdf/arm/scara.urdf.xacro"/>
+    <xacro:include filename="$(find robot_model_description)/urdf/arm/gripper.urdf.xacro"/>
+    <xacro:include filename="$(find robot_model_description)/urdf/ros2_control.urdf.xacro"/>
+    <xacro:include filename="$(find robot_model_description)/urdf/utils/utils.urdf.xacro"/>
+    <xacro:include filename="$(find robot_model_description)/urdf/sensors/camera.urdf.xacro"/>
+    <xacro:include filename="$(find robot_model_description)/urdf/sensors/imu_sensor.urdf.xacro"/>
+    <xacro:include filename="$(find robot_model_description)/urdf/sensors/sensors.urdf.xacro"/>
     <!-- properties -->
     <xacro:property name="PI" value="3.1415926535897931"/>
@@ -36,7 +36,7 @@
     <xacro:imu_sensor parent="arm_gripper_link"/>
     <!-- gazebo ROS control plugins -->
-    <xacro:include filename="$(find robot_description)/urdf/ros2_control.urdf.xacro"/>
-    <xacro:arg name="config_controllers" default="$(find robot_description)/config/rover_controllers.yaml"/>
+    <xacro:include filename="$(find robot_model_description)/urdf/ros2_control.urdf.xacro"/>
+    <xacro:arg name="config_controllers" default="$(find robot_model_description)/config/rover_controllers.yaml"/>
     <xacro:arg name="update_rate" default="20"/>
-    <xacro:ros2_control/>
+    <!-- <xacro:ros2_control/> -->
 </robot>

File: Prácticas/Práctica 3: Simulación de Robots usando Middleware/src/robot_model_description/urdf/arm/gripper.urdf.xacro (robot description, xacro)
@@ -20,5 +20,5 @@
         <origin rpy="3.14159 0.00000 3.14159" xyz="1.05643 0.00000 0.00000"/>
         <geometry>
-          <mesh filename="file://$(find robot_description)/meshes/dae/Cube.009.dae" scale="0.30000 0.15000 0.02500"/>
+          <mesh filename="file://$(find robot_model_description)/meshes/dae/Cube.009.dae" scale="0.30000 0.15000 0.02500"/>
         </geometry>
       </collision>
@@ -32,5 +32,5 @@
         <material name="yellow.001"/>
         <geometry>
-          <mesh filename="file://$(find robot_description)/meshes/dae/Cube.009.dae" scale="0.30000 0.15000 0.02500"/>
+          <mesh filename="file://$(find robot_model_description)/meshes/dae/Cube.009.dae" scale="0.30000 0.15000 0.02500"/>
         </geometry>
       </visual>
@@ -40,5 +40,5 @@
         <origin rpy="0.00000 0.00000 0.00000" xyz="-1.05643 0.00000 0.00000"/>
         <geometry>
-          <mesh filename="file://$(find robot_description)/meshes/dae/Cube.008.dae" scale="0.30000 0.15000 0.02500"/>
+          <mesh filename="file://$(find robot_model_description)/meshes/dae/Cube.008.dae" scale="0.30000 0.15000 0.02500"/>
         </geometry>
       </collision>
@@ -52,5 +52,5 @@
         <material name="yellow.001"/>
         <geometry>
-          <mesh filename="file://$(find robot_description)/meshes/dae/Cube.008.dae" scale="0.30000 0.15000 0.02500"/>
+          <mesh filename="file://$(find robot_model_description)/meshes/dae/Cube.008.dae" scale="0.30000 0.15000 0.02500"/>
         </geometry>
       </visual>

File: Prácticas/Práctica 3: Simulación de Robots usando Middleware/src/robot_model_description/urdf/arm/scara.urdf.xacro (robot description, xacro)
@@ -39,5 +39,5 @@
         <origin rpy="0.00000 0.00000 0.00000" xyz="0.00000 -0.50000 0.00000"/>
         <geometry>
-          <mesh filename="file://$(find robot_description)/meshes/dae/Cylinder.015.dae" scale="0.20000 0.20000 0.10000"/>
+          <mesh filename="file://$(find robot_model_description)/meshes/dae/Cylinder.015.dae" scale="0.20000 0.20000 0.10000"/>
         </geometry>
       </collision>
@@ -51,5 +51,5 @@
         <material name="yellow.001"/>
         <geometry>
-          <mesh filename="file://$(find robot_description)/meshes/dae/Cylinder.015.dae" scale="0.20000 0.20000 0.10000"/>
+          <mesh filename="file://$(find robot_model_description)/meshes/dae/Cylinder.015.dae" scale="0.20000 0.20000 0.10000"/>
         </geometry>
       </visual>
@@ -59,5 +59,5 @@
         <origin rpy="0.00000 0.00000 0.00000" xyz="0.00000 -0.50000 0.00000"/>
         <geometry>
-          <mesh filename="file://$(find robot_description)/meshes/dae/Cylinder.017.dae" scale="0.20000 0.20000 0.10000"/>
+          <mesh filename="file://$(find robot_model_description)/meshes/dae/Cylinder.017.dae" scale="0.20000 0.20000 0.10000"/>
         </geometry>
       </collision>
@@ -71,5 +71,5 @@
         <material name="yellow.001"/>
         <geometry>
-          <mesh filename="file://$(find robot_description)/meshes/dae/Cylinder.017.dae" scale="0.20000 0.20000 0.10000"/>
+          <mesh filename="file://$(find robot_model_description)/meshes/dae/Cylinder.017.dae" scale="0.20000 0.20000 0.10000"/>
         </geometry>
       </visual>
@@ -119,5 +119,5 @@
         <origin rpy="0.00000 0.00000 0.00000" xyz="0.00000 0.00000 0.00003"/>
         <geometry>
-          <mesh filename="file://$(find robot_description)/meshes/dae/Cube.007.dae" scale="0.35000 0.15000 0.02500"/>
+          <mesh filename="file://$(find robot_model_description)/meshes/dae/Cube.007.dae" scale="0.35000 0.15000 0.02500"/>
         </geometry>
       </collision>
@@ -131,5 +131,5 @@
         <material name="yellow.001"/>
         <geometry>
-          <mesh filename="file://$(find robot_description)/meshes/dae/Cube.007.dae" scale="0.35000 0.15000 0.02500"/>
+          <mesh filename="file://$(find robot_model_description)/meshes/dae/Cube.007.dae" scale="0.35000 0.15000 0.02500"/>
         </geometry>
       </visual>

File: Prácticas/Práctica 3: Simulación de Robots usando Middleware/src/robot_model_description/urdf/base/robot_base.urdf.xacro (robot description, xacro)
@@ -43,5 +43,5 @@
         <material name="red.001"/>
         <geometry>
-          <mesh filename="file://$(find robot_description)/meshes/dae/Cube.003.dae" scale="0.05000 1.00000 0.35000"/>
+          <mesh filename="file://$(find robot_model_description)/meshes/dae/Cube.003.dae" scale="0.05000 1.00000 0.35000"/>
         </geometry>
       </visual>

File: Prácticas/Práctica 3: Simulación de Robots usando Middleware/src/robot_model_description/urdf/wheels/rover_wheel.urdf.xacro (robot description, xacro)
@@ -54,5 +54,5 @@
         <origin rpy="0.00000 1.57080 0.00000" xyz="0.00000 0.00000 0.00000"/>
         <geometry>
-          <mesh filename="file://$(find robot_description)/meshes/dae/Cylinder.009.dae" scale="0.05000 0.05000 0.20000"/>
+          <mesh filename="file://$(find robot_model_description)/meshes/dae/Cylinder.009.dae" scale="0.05000 0.05000 0.20000"/>
         </geometry>
         <!--
@@ -79,5 +79,5 @@
         <material name="black.007"/>
         <geometry>
-          <mesh filename="file://$(find robot_description)/meshes/dae/Cylinder.009.dae" scale="0.05000 0.05000 0.20000"/>
+          <mesh filename="file://$(find robot_model_description)/meshes/dae/Cylinder.009.dae" scale="0.05000 0.05000 0.20000"/>
         </geometry>
       </visual>
@@ -87,5 +87,5 @@
         <origin rpy="0.00000 1.57080 0.00000" xyz="0.00000 0.00000 0.00000"/>
         <geometry>
-          <mesh filename="file://$(find robot_description)/meshes/dae/Cylinder.004.dae" scale="0.05000 0.05000 0.20000"/>
+          <mesh filename="file://$(find robot_model_description)/meshes/dae/Cylinder.004.dae" scale="0.05000 0.05000 0.20000"/>
         </geometry>
       </collision>
@@ -99,5 +99,5 @@
         <material name="black.007"/>
         <geometry>
-          <mesh filename="file://$(find robot_description)/meshes/dae/Cylinder.004.dae" scale="0.05000 0.05000 0.20000"/>
+          <mesh filename="file://$(find robot_model_description)/meshes/dae/Cylinder.004.dae" scale="0.05000 0.05000 0.20000"/>
         </geometry>
       </visual>
@@ -107,5 +107,5 @@
         <origin rpy="0.00000 1.57080 0.00000" xyz="0.00000 0.00000 0.00000"/>
         <geometry>
-          <mesh filename="file://$(find robot_description)/meshes/dae/Cylinder.010.dae" scale="0.05000 0.05000 0.20000"/>
+          <mesh filename="file://$(find robot_model_description)/meshes/dae/Cylinder.010.dae" scale="0.05000 0.05000 0.20000"/>
         </geometry>
       </collision>
@@ -119,5 +119,5 @@
         <material name="black.007"/>
         <geometry>
-          <mesh filename="file://$(find robot_description)/meshes/dae/Cylinder.010.dae" scale="0.05000 0.05000 0.20000"/>
+          <mesh filename="file://$(find robot_model_description)/meshes/dae/Cylinder.010.dae" scale="0.05000 0.05000 0.20000"/>
         </geometry>
       </visual>
@@ -127,5 +127,5 @@
         <origin rpy="0.00000 1.57080 0.00000" xyz="0.00000 0.00000 0.00000"/>
         <geometry>
-          <mesh filename="file://$(find robot_description)/meshes/dae/Cylinder.011.dae" scale="0.05000 0.05000 0.20000"/>
+          <mesh filename="file://$(find robot_model_description)/meshes/dae/Cylinder.011.dae" scale="0.05000 0.05000 0.20000"/>
         </geometry>
       </collision>
@@ -139,5 +139,5 @@
         <material name="black.007"/>
         <geometry>
-          <mesh filename="file://$(find robot_description)/meshes/dae/Cylinder.011.dae" scale="0.05000 0.05000 0.20000"/>
+          <mesh filename="file://$(find robot_model_description)/meshes/dae/Cylinder.011.dae" scale="0.05000 0.05000 0.20000"/>
         </geometry>
       </visual>
@@ -147,5 +147,5 @@
         <origin rpy="0.00000 -1.57080 0.00000" xyz="0.00000 0.00000 0.00000"/>
         <geometry>
-          <mesh filename="file://$(find robot_description)/meshes/dae/Cylinder.002.dae" scale="0.05000 0.05000 0.20000"/>
+          <mesh filename="file://$(find robot_model_description)/meshes/dae/Cylinder.002.dae" scale="0.05000 0.05000 0.20000"/>
         </geometry>
       </collision>
@@ -159,5 +159,5 @@
         <material name="black.007"/>
         <geometry>
-          <mesh filename="file://$(find robot_description)/meshes/dae/Cylinder.002.dae" scale="0.05000 0.05000 0.20000"/>
+          <mesh filename="file://$(find robot_model_description)/meshes/dae/Cylinder.002.dae" scale="0.05000 0.05000 0.20000"/>
         </geometry>
       </visual>
@@ -167,5 +167,5 @@
         <origin rpy="0.00000 -1.57080 0.00000" xyz="0.00000 0.00000 0.00000"/>
         <geometry>
-          <mesh filename="file://$(find robot_description)/meshes/dae/Cylinder.003.dae" scale="0.05000 0.05000 0.20000"/>
+          <mesh filename="file://$(find robot_model_description)/meshes/dae/Cylinder.003.dae" scale="0.05000 0.05000 0.20000"/>
         </geometry>
       </collision>
@@ -179,5 +179,5 @@
         <material name="black.007"/>
         <geometry>
-          <mesh filename="file://$(find robot_description)/meshes/dae/Cylinder.003.dae" scale="0.05000 0.05000 0.20000"/>
+          <mesh filename="file://$(find robot_model_description)/meshes/dae/Cylinder.003.dae" scale="0.05000 0.05000 0.20000"/>
         </geometry>
       </visual>
@@ -187,5 +187,5 @@
         <origin rpy="0.00000 -1.57080 0.00000" xyz="0.00000 0.00000 0.00000"/>
         <geometry>
-          <mesh filename="file://$(find robot_description)/meshes/dae/Cylinder.001.dae" scale="0.05000 0.05000 0.20000"/>
+          <mesh filename="file://$(find robot_model_description)/meshes/dae/Cylinder.001.dae" scale="0.05000 0.05000 0.20000"/>
         </geometry>
       </collision>
@@ -199,5 +199,5 @@
         <material name="black.007"/>
         <geometry>
-          <mesh filename="file://$(find robot_description)/meshes/dae/Cylinder.001.dae" scale="0.05000 0.05000 0.20000"/>
+          <mesh filename="file://$(find robot_model_description)/meshes/dae/Cylinder.001.dae" scale="0.05000 0.05000 0.20000"/>
         </geometry>
       </visual>
@@ -207,5 +207,5 @@
         <origin rpy="0.00000 -1.57080 0.00000" xyz="0.00000 0.00000 0.00000"/>
         <geometry>
-          <mesh filename="file://$(find robot_description)/meshes/dae/Cylinder.dae" scale="0.05000 0.05000 0.20000"/>
+          <mesh filename="file://$(find robot_model_description)/meshes/dae/Cylinder.dae" scale="0.05000 0.05000 0.20000"/>
         </geometry>
       </collision>
@@ -219,5 +219,5 @@
         <material name="black.007"/>
         <geometry>
-          <mesh filename="file://$(find robot_description)/meshes/dae/Cylinder.dae" scale="0.05000 0.05000 0.20000"/>
+          <mesh filename="file://$(find robot_model_description)/meshes/dae/Cylinder.dae" scale="0.05000 0.05000 0.20000"/>
         </geometry>
       </visual>
