Commit message: UPLOADING FILES ...

File: Prácticas/Práctica 3: Simulación de Robots usando Middleware/src/robot_model_description/robots/robot.urdf.xacro (robot description, xacro)
@@ -13,10 +13,4 @@
     <!-- properties -->
     <xacro:property name="PI" value="3.1415926535897931"/>
-    <xacro:property name="wheel_offset_x" value="0.95"/>
-    <xacro:property name="wheel_offset_y" value="0.95"/>
-    <xacro:property name="wheel_offset_z" value="-0.38"/>
-    <xacro:property name="arm_offset_x" value="0.0"/>
-    <xacro:property name="arm_offset_y" value="0.82"/>
-    <xacro:property name="arm_offset_z" value="0.69"/>
     <!-- arguments -->
     <xacro:arg name="robot_ns" default=""/>
@@ -27,16 +21,15 @@
     <xacro:robot_base/>
     <!-- wheels -->
-    <xacro:rover_wheel parent="Base_link"/>
+    <xacro:rover_wheel parent="base_link"/>
     <!-- arm -->
-    <xacro:scara parent="Base_link"/>
+    <xacro:scara parent="base_link"/>
     <xacro:gripper parent="arm_gripper_link"/>
     <!-- sensors -->
-    <xacro:camera parent="Base_link"/>
+    <xacro:camera parent="base_link"/>
     <xacro:sensors parent="arm_gripper_link"/>
-    <xacro:imu_sensor parent="arm_gripper_link"/>
+    <xacro:imu_sensor parent="base_link"/>
     <!-- gazebo ROS control plugins -->
-    <xacro:include filename="$(find robot_model_description)/urdf/ros2_control.urdf.xacro"/>
     <xacro:arg name="config_controllers" default="$(find robot_model_description)/config/rover_controllers.yaml"/>
-    <xacro:arg name="update_rate" default="20"/>
+    <xacro:arg name="update_rate" default="30"/>
     <xacro:ros2_control/>
 </robot>

File: Prácticas/Práctica 3: Simulación de Robots usando Middleware/src/robot_model_description/urdf/arm/gripper.urdf.xacro (robot description, xacro)
@@ -3,5 +3,5 @@
   <xacro:macro name="gripper"  params="parent" >
     <joint name="gripper_left_link_joint" type="prismatic">
-      <limit lower="0.00000" upper="0.15000" effort="0.00000" velocity="0.00000"/>
+      <limit lower="0.00000" upper="0.15000" effort="1000.00000" velocity="100.00000"/>
       <origin rpy="0.00000 -1.57080 0.00000" xyz="0.32000 0.00000 -2.53589"/>
       <parent link="${parent}"/>
@@ -10,5 +10,5 @@
     </joint>
     <joint name="gripper_right_link_joint" type="prismatic">
-      <limit lower="0.00000" upper="0.15000" effort="0.00000" velocity="0.00000"/>
+      <limit lower="0.00000" upper="0.15000" effort="1000.00000" velocity="100.00000"/>
       <origin rpy="0.00000 1.57080 0.00000" xyz="-0.32000 0.00000 -2.53589"/>
       <parent link="${parent}"/>

File: Prácticas/Práctica 3: Simulación de Robots usando Middleware/src/robot_model_description/urdf/arm/scara.urdf.xacro (robot description, xacro)
@@ -3,5 +3,5 @@
   <xacro:macro name="scara" params="parent" >
     <joint name="arm_1_link_joint" type="continuous">
-      <limit lower="0" upper="0" effort="0.00000" velocity="0.00000"/>
+      <limit lower="0" upper="0" effort="1000.00000" velocity="100.00000"/>
       <origin rpy="0.00000 0.00000 0.00000" xyz="0.00000 0.00000 0.65000"/>
       <parent link="arm_column_link"/>
@@ -10,5 +10,5 @@
     </joint>
     <joint name="arm_2_link_joint" type="continuous">
-      <limit lower="0" upper="0" effort="0.00000" velocity="0.00000"/>
+      <limit lower="0" upper="0" effort="1000.00000" velocity="100.00000"/>
       <origin rpy="0.00000 0.00000 0.00000" xyz="0.00000 -1.00000 0.20000"/>
       <parent link="arm_1_link"/>
@@ -18,9 +18,9 @@
     <joint name="arm_base_link_joint" type="fixed">
       <origin rpy="0.00000 0.00000 0.00000" xyz="0.00000 -1.08925 0.52413"/>
-      <parent link="Base_link"/>
+      <parent link="base_link"/>
       <child link="arm_base_link"/>
     </joint>
     <joint name="arm_column_link_joint" type="continuous">
-      <limit lower="0" upper="0" effort="0.00000" velocity="0.00000"/>
+      <limit lower="0" upper="0" effort="1000.00000" velocity="100.00000"/>
       <origin rpy="0.00000 0.00000 0.00000" xyz="0.00000 0.00000 0.85000"/>
       <parent link="arm_base_link"/>
@@ -29,5 +29,5 @@
     </joint>
     <joint name="arm_gripper_link_joint" type="prismatic">
-      <limit lower="-1.25000" upper="1.00000" effort="0.00000" velocity="0.00000"/>
+      <limit lower="-1.25000" upper="1.00000" effort="1000.00000" velocity="100.00000"/>
       <origin rpy="0.00000 0.00000 0.00000" xyz="0.00000 -1.00000 -0.07053"/>
       <parent link="arm_2_link"/>

File: Prácticas/Práctica 3: Simulación de Robots usando Middleware/src/robot_model_description/urdf/base/robot_base.urdf.xacro (robot description, xacro)
@@ -2,30 +2,30 @@
 <robot name="robot_model" xmlns:xacro="http://wiki.ros.org/xacro">
   <xacro:macro name="robot_base" >
-    <joint name="Base_link_joint" type="fixed">
+    <joint name="base_link_joint" type="fixed">
       <origin rpy="0.00000 0.00000 0.00000" xyz="0.00000 0.00000 1.00000"/>
       <parent link="base_footprint"/>
-      <child link="Base_link"/>
+      <child link="base_link"/>
     </joint>
     <joint name="box_down_side_link_joint" type="fixed">
       <origin rpy="0.00000 0.00000 1.57080" xyz="0.00000 1.86075 0.77413"/>
-      <parent link="Base_link"/>
+      <parent link="base_link"/>
       <child link="box_down_side_link"/>
     </joint>
     <joint name="box_left_side_link_joint" type="fixed">
       <origin rpy="0.00000 0.00000 0.00000" xyz="0.45000 0.91075 0.77413"/>
-      <parent link="Base_link"/>
+      <parent link="base_link"/>
       <child link="box_left_side_link"/>
     </joint>
     <joint name="box_right_side_link_joint" type="fixed">
       <origin rpy="0.00000 0.00000 0.00000" xyz="-0.45000 0.91075 0.77413"/>
-      <parent link="Base_link"/>
+      <parent link="base_link"/>
       <child link="box_right_side_link"/>
     </joint>
     <joint name="box_up_side_link_joint" type="fixed">
       <origin rpy="0.00000 0.00000 1.57080" xyz="0.00000 -0.03925 0.77413"/>
-      <parent link="Base_link"/>
+      <parent link="base_link"/>
       <child link="box_up_side_link"/>
     </joint>
-    <link name="Base_link">
+    <link name="base_link">
       <collision name="Base_collision">
         <origin rpy="0.00000 0.00000 0.00000" xyz="0.00000 -0.09000 -0.07000"/>
@@ -127,5 +127,19 @@
       </visual>
     </link>
-    <link name="base_footprint"/>
+    <link name="base_footprint">
+      <collision name="base_footprint_collision">
+        <origin rpy="0.00000 0.00000 0.00000" xyz="0.00000 0.00000 0.00000"/>
+        <geometry>
+          <box size="0.10000 0.10000 0.10000"/>
+        </geometry>
+      </collision>
+      <visual name="base_footprint">
+        <origin rpy="0.00000 0.00000 0.00000" xyz="0.00000 0.00000 0.00000"/>
+        <material name="red.001"/>
+        <geometry>
+          <box size="0.10000 0.10000 0.10000"/>
+        </geometry>
+      </visual>
+    </link>
   </xacro:macro>
 </robot>

File: Prácticas/Práctica 3: Simulación de Robots usando Middleware/src/robot_model_description/urdf/ros2_control.urdf.xacro (robot description, xacro)
@@ -3,6 +3,17 @@
   <xacro:macro name="ros2_control">
     <gazebo>
-      <plugin filename="libgz_ros2_control-system.so" name="gz_ros2_control::GazeboSimROS2ControlPlugin">
+      <plugin filename="libgz_ros2_control-system.so"
+              name="gz_ros2_control::GazeboSimROS2ControlPlugin">
         <parameters>$(arg config_controllers)</parameters>
+      </plugin>
+      <plugin name="libgazebo_ros_diff_drive.so"
+              filename="gazebo_ros_diff_drive">
+      <ros>
+        <remapping>cmd_vel:=/cmd_vel</remapping>
+      </ros>
+      <left_joint>wheel_down_left_link_joint</left_joint>
+      <right_joint>wheel_down_right_link_joint</right_joint>
+      <wheel_separation>1.5</wheel_separation>
+      <wheel_radius>0.3</wheel_radius>
       </plugin>
     </gazebo>
@@ -11,4 +22,6 @@
         <plugin>gz_ros2_control/GazeboSimSystem</plugin>
       </hardware>
+      <!-- Interfaces de las articulaciones -->
+      <!-- Rueda delantera izquierda -->
       <joint name="wheel_up_left_link_joint">
         <command_interface name="velocity">
@@ -20,4 +33,5 @@
         <state_interface name="effort"/>
       </joint>
+      <!-- Rueda delantera derecha -->
       <joint name="wheel_up_right_link_joint">
         <command_interface name="velocity">
@@ -29,4 +43,5 @@
         <state_interface name="effort"/>
       </joint>
+      <!-- Rueda trasera izquierda -->
       <joint name="wheel_down_left_link_joint">
         <command_interface name="velocity">
@@ -38,4 +53,5 @@
         <state_interface name="effort"/>
       </joint>
+      <!-- Rueda trasera derecha -->
       <joint name="wheel_down_right_link_joint">
         <command_interface name="velocity">

File: Prácticas/Práctica 3: Simulación de Robots usando Middleware/src/robot_model_description/urdf/sensors/camera.urdf.xacro (robot description, xacro)
@@ -8,4 +8,10 @@
     </joint>
     <link name="camera_link">
+      <collision name="camera_collision">
+        <origin rpy="0.00000 0.00000 0.00000" xyz="0.00000 0.00000 0.00000"/>
+        <geometry>
+          <box size="0.10000 0.30000 0.20000"/>
+        </geometry>
+      </collision>
       <visual name="camera">
         <origin rpy="0.00000 0.00000 0.00000" xyz="0.00000 0.00000 -0.20000"/>

File: Prácticas/Práctica 3: Simulación de Robots usando Middleware/src/robot_model_description/urdf/sensors/imu_sensor.urdf.xacro (robot description, xacro)
@@ -8,4 +8,10 @@
     </joint>
     <link name="IMU_link">
+      <collision name="IMU_collision">
+        <origin rpy="0.00000 0.00000 0.00000" xyz="0.00000 0.00000 0.00000"/>
+        <geometry>
+            <box size="0.10000 0.10000 0.10000"/>
+        </geometry>
+      </collision>
       <visual name="IMU">
         <origin rpy="0.00000 0.00000 0.00000" xyz="0.00000 0.00000 0.00000"/>

File: Prácticas/Práctica 3: Simulación de Robots usando Middleware/src/robot_model_description/urdf/sensors/sensors.urdf.xacro (robot description, xacro)
@@ -8,4 +8,10 @@
     </joint>
     <link name="sensors_link">
+      <collision name="sensors_collision">
+        <origin rpy="0.00000 0.00000 0.00000" xyz="0.00000 0.00000 0.00000"/>
+        <geometry>
+          <box size="0.10000 0.30000 0.20000"/>
+        </geometry>
+      </collision>
       <visual name="sensors">
         <origin rpy="0.00000 0.00000 0.00000" xyz="0.00000 0.00000 0.00000"/>
@@ -15,4 +21,9 @@
         </geometry>
       </visual>
+      <inertial>
+        <mass value="1.0"/>
+        <origin xyz="0 0 0"/>
+        <inertia ixx="0.1" ixy="0" ixz="0" iyy="0.1" iyz="0" izz="0.1"/>
+      </inertial>
     </link>
     <gazebo reference="sensors_link">
