Commit message: UPLOADING FILES ...

File: Prácticas/Práctica 3: Simulación de Robots usando Middleware/src/robot_model_description/urdf/wheels/rover_wheel.urdf.xacro (robot description, xacro)
@@ -4,24 +4,24 @@
     <joint name="subjection_down_left_wheel_link_joint" type="fixed">
       <origin rpy="0.00000 0.00000 0.00000" xyz="0.53571 0.91075 -0.81158"/>
-      <parent link="Base_link"/>
+      <parent link="base_link"/>
       <child link="subjection_down_left_wheel_link"/>
     </joint>
     <joint name="subjection_down_right_wheel_link_joint" type="fixed">
       <origin rpy="0.00000 0.00000 0.00000" xyz="-0.53571 0.91075 -0.81158"/>
-      <parent link="Base_link"/>
+      <parent link="base_link"/>
       <child link="subjection_down_right_wheel_link"/>
     </joint>
     <joint name="subjection_up_left_wheel_link_joint" type="fixed">
       <origin rpy="0.00000 0.00000 0.00000" xyz="0.53571 -1.08925 -0.81158"/>
-      <parent link="Base_link"/>
+      <parent link="base_link"/>
       <child link="subjection_up_left_wheel_link"/>
     </joint>
     <joint name="subjection_up_right_wheel_link_joint" type="fixed">
       <origin rpy="0.00000 0.00000 0.00000" xyz="-0.53571 -1.08925 -0.81158"/>
-      <parent link="Base_link"/>
+      <parent link="base_link"/>
       <child link="subjection_up_right_wheel_link"/>
     </joint>
     <joint name="wheel_down_left_link_joint" type="continuous">
-      <limit lower="0" upper="0" effort="0.00000" velocity="0.00000"/>
+      <limit lower="0" upper="0" effort="1000.00000" velocity="100.00000"/>
       <origin rpy="0.00000 1.57080 0.00000" xyz="0.26429 0.00000 -0.06429"/>
       <parent link="subjection_down_left_wheel_link"/>
@@ -30,5 +30,5 @@
     </joint>
     <joint name="wheel_down_right_link_joint" type="continuous">
-      <limit lower="0" upper="0" effort="0.00000" velocity="0.00000"/>
+      <limit lower="0" upper="0" effort="1000.00000" velocity="100.00000"/>
       <origin rpy="0.00000 1.57080 0.00000" xyz="-0.26429 0.00000 -0.06429"/>
       <parent link="subjection_down_right_wheel_link"/>
@@ -37,5 +37,5 @@
     </joint>
     <joint name="wheel_up_left_link_joint" type="continuous">
-      <limit lower="0" upper="0" effort="0.00000" velocity="0.00000"/>
+      <limit lower="0" upper="0" effort="1000.00000" velocity="100.00000"/>
       <origin rpy="0.00000 1.57080 0.00000" xyz="0.26429 0.00000 -0.06429"/>
       <parent link="subjection_up_left_wheel_link"/>
@@ -44,5 +44,5 @@
     </joint>
     <joint name="wheel_up_right_link_joint" type="continuous">
-      <limit lower="0" upper="0" effort="0.00000" velocity="0.00000"/>
+      <limit lower="0" upper="0" effort="1000.00000" velocity="100.00000"/>
       <origin rpy="0.00000 1.57080 0.00000" xyz="-0.26429 0.00000 -0.06429"/>
       <parent link="subjection_up_right_wheel_link"/>
@@ -56,5 +56,84 @@
           <mesh filename="file://$(find robot_model_description)/meshes/dae/Cylinder.009.dae" scale="0.05000 0.05000 0.20000"/>
         </geometry>
-        <!--
+      </collision>
+      <inertial>
+        <inertia ixx="0.09178" ixy="0.00000" ixz="0.05238" iyy="0.21726" iyz="0.00000" izz="0.13657"/>
+        <origin rpy="0.00000 0.00000 0.00000" xyz="0.00000 0.00000 0.00000"/>
+        <mass value="10.00000"/>
+      </inertial>
+      <visual name="subjection_down_left_wheel">
+        <origin rpy="0.00000 1.57080 0.00000" xyz="0.00000 0.00000 0.00000"/>
+        <material name="black.007"/>
+        <geometry>
+          <mesh filename="file://$(find robot_model_description)/meshes/dae/Cylinder.009.dae" scale="0.05000 0.05000 0.20000"/>
+        </geometry>
+      </visual>
+    </link>
+    <link name="subjection_down_right_wheel_link">
+      <collision name="subjection_down_right_wheel_collision">
+        <origin rpy="0.00000 1.57080 0.00000" xyz="0.00000 0.00000 0.00000"/>
+        <geometry>
+          <mesh filename="file://$(find robot_model_description)/meshes/dae/Cylinder.004.dae" scale="0.05000 0.05000 0.20000"/>
+        </geometry>
+      </collision>
+      <inertial>
+        <inertia ixx="0.09178" ixy="0.00000" ixz="-0.05238" iyy="0.21726" iyz="0.00000" izz="0.13657"/>
+        <origin rpy="0.00000 0.00000 0.00000" xyz="0.00000 0.00000 0.00000"/>
+        <mass value="10.00000"/>
+      </inertial>
+      <visual name="subjection_down_right_wheel">
+        <origin rpy="0.00000 1.57080 0.00000" xyz="0.00000 0.00000 0.00000"/>
+        <material name="black.007"/>
+        <geometry>
+          <mesh filename="file://$(find robot_model_description)/meshes/dae/Cylinder.004.dae" scale="0.05000 0.05000 0.20000"/>
+        </geometry>
+      </visual>
+    </link>
+    <link name="subjection_up_left_wheel_link">
+      <collision name="subjection_up_left_wheel_collision">
+        <origin rpy="0.00000 1.57080 0.00000" xyz="0.00000 0.00000 0.00000"/>
+        <geometry>
+          <mesh filename="file://$(find robot_model_description)/meshes/dae/Cylinder.010.dae" scale="0.05000 0.05000 0.20000"/>
+        </geometry>
+      </collision>
+      <inertial>
+        <inertia ixx="0.09178" ixy="0.00000" ixz="0.05238" iyy="0.21726" iyz="0.00000" izz="0.13657"/>
+        <origin rpy="0.00000 0.00000 0.00000" xyz="0.00000 0.00000 0.00000"/>
+        <mass value="10.00000"/>
+      </inertial>
+      <visual name="subjection_up_left_wheel">
+        <origin rpy="0.00000 1.57080 0.00000" xyz="0.00000 0.00000 0.00000"/>
+        <material name="black.007"/>
+        <geometry>
+          <mesh filename="file://$(find robot_model_description)/meshes/dae/Cylinder.010.dae" scale="0.05000 0.05000 0.20000"/>
+        </geometry>
+      </visual>
+    </link>
+    <link name="subjection_up_right_wheel_link">
+      <collision name="subjection_up_right_wheel_collision">
+        <origin rpy="0.00000 1.57080 0.00000" xyz="0.00000 0.00000 0.00000"/>
+        <geometry>
+          <mesh filename="file://$(find robot_model_description)/meshes/dae/Cylinder.011.dae" scale="0.05000 0.05000 0.20000"/>
+        </geometry>
+      </collision>
+      <inertial>
+        <inertia ixx="0.09178" ixy="0.00000" ixz="-0.05238" iyy="0.21726" iyz="0.00000" izz="0.13657"/>
+        <origin rpy="0.00000 0.00000 0.00000" xyz="0.00000 0.00000 0.00000"/>
+        <mass value="10.00000"/>
+      </inertial>
+      <visual name="subjection_up_right_wheel">
+        <origin rpy="0.00000 1.57080 0.00000" xyz="0.00000 0.00000 0.00000"/>
+        <material name="black.007"/>
+        <geometry>
+          <mesh filename="file://$(find robot_model_description)/meshes/dae/Cylinder.011.dae" scale="0.05000 0.05000 0.20000"/>
+        </geometry>
+      </visual>
+    </link>
+    <link name="wheel_down_left_link">
+      <collision name="wheel_down_left_collision">
+        <origin rpy="0.00000 -1.57080 0.00000" xyz="0.00000 0.00000 0.00000"/>
+        <geometry>
+          <mesh filename="file://$(find robot_model_description)/meshes/dae/Cylinder.002.dae" scale="0.05000 0.05000 0.20000"/>
+        </geometry>
         <surface>
           <friction>
@@ -62,91 +141,7 @@
               <mu>1.000000</mu>
               <mu2>1.000000</mu2>
-              <fdir1>0.000000 0.000000 1.000000</fdir1>
-              <slip1>0.500000</slip1>
-              <slip2>0.500000</slip2>
             </ode>
           </friction>
         </surface>
-        -->
-      </collision>
-      <inertial>
-        <inertia ixx="0.09178" ixy="0.00000" ixz="0.05238" iyy="0.21726" iyz="0.00000" izz="0.13657"/>
-        <origin rpy="0.00000 0.00000 0.00000" xyz="0.00000 0.00000 0.00000"/>
-        <mass value="10.00000"/>
-      </inertial>
-      <visual name="subjection_down_left_wheel">
-        <origin rpy="0.00000 1.57080 0.00000" xyz="0.00000 0.00000 0.00000"/>
-        <material name="black.007"/>
-        <geometry>
-          <mesh filename="file://$(find robot_model_description)/meshes/dae/Cylinder.009.dae" scale="0.05000 0.05000 0.20000"/>
-        </geometry>
-      </visual>
-    </link>
-    <link name="subjection_down_right_wheel_link">
-      <collision name="subjection_down_right_wheel_collision">
-        <origin rpy="0.00000 1.57080 0.00000" xyz="0.00000 0.00000 0.00000"/>
-        <geometry>
-          <mesh filename="file://$(find robot_model_description)/meshes/dae/Cylinder.004.dae" scale="0.05000 0.05000 0.20000"/>
-        </geometry>
-      </collision>
-      <inertial>
-        <inertia ixx="0.09178" ixy="0.00000" ixz="-0.05238" iyy="0.21726" iyz="0.00000" izz="0.13657"/>
-        <origin rpy="0.00000 0.00000 0.00000" xyz="0.00000 0.00000 0.00000"/>
-        <mass value="10.00000"/>
-      </inertial>
-      <visual name="subjection_down_right_wheel">
-        <origin rpy="0.00000 1.57080 0.00000" xyz="0.00000 0.00000 0.00000"/>
-        <material name="black.007"/>
-        <geometry>
-          <mesh filename="file://$(find robot_model_description)/meshes/dae/Cylinder.004.dae" scale="0.05000 0.05000 0.20000"/>
-        </geometry>
-      </visual>
-    </link>
-    <link name="subjection_up_left_wheel_link">
-      <collision name="subjection_up_left_wheel_collision">
-        <origin rpy="0.00000 1.57080 0.00000" xyz="0.00000 0.00000 0.00000"/>
-        <geometry>
-          <mesh filename="file://$(find robot_model_description)/meshes/dae/Cylinder.010.dae" scale="0.05000 0.05000 0.20000"/>
-        </geometry>
-      </collision>
-      <inertial>
-        <inertia ixx="0.09178" ixy="0.00000" ixz="0.05238" iyy="0.21726" iyz="0.00000" izz="0.13657"/>
-        <origin rpy="0.00000 0.00000 0.00000" xyz="0.00000 0.00000 0.00000"/>
-        <mass value="10.00000"/>
-      </inertial>
-      <visual name="subjection_up_left_wheel">
-        <origin rpy="0.00000 1.57080 0.00000" xyz="0.00000 0.00000 0.00000"/>
-        <material name="black.007"/>
-        <geometry>
-          <mesh filename="file://$(find robot_model_description)/meshes/dae/Cylinder.010.dae" scale="0.05000 0.05000 0.20000"/>
-        </geometry>
-      </visual>
-    </link>
-    <link name="subjection_up_right_wheel_link">
-      <collision name="subjection_up_right_wheel_collision">
-        <origin rpy="0.00000 1.57080 0.00000" xyz="0.00000 0.00000 0.00000"/>
-        <geometry>
-          <mesh filename="file://$(find robot_model_description)/meshes/dae/Cylinder.011.dae" scale="0.05000 0.05000 0.20000"/>
-        </geometry>
-      </collision>
-      <inertial>
-        <inertia ixx="0.09178" ixy="0.00000" ixz="-0.05238" iyy="0.21726" iyz="0.00000" izz="0.13657"/>
-        <origin rpy="0.00000 0.00000 0.00000" xyz="0.00000 0.00000 0.00000"/>
-        <mass value="10.00000"/>
-      </inertial>
-      <visual name="subjection_up_right_wheel">
-        <origin rpy="0.00000 1.57080 0.00000" xyz="0.00000 0.00000 0.00000"/>
-        <material name="black.007"/>
-        <geometry>
-          <mesh filename="file://$(find robot_model_description)/meshes/dae/Cylinder.011.dae" scale="0.05000 0.05000 0.20000"/>
-        </geometry>
-      </visual>
-    </link>
-    <link name="wheel_down_left_link">
-      <collision name="wheel_down_left_collision">
-        <origin rpy="0.00000 -1.57080 0.00000" xyz="0.00000 0.00000 0.00000"/>
-        <geometry>
-          <mesh filename="file://$(find robot_model_description)/meshes/dae/Cylinder.002.dae" scale="0.05000 0.05000 0.20000"/>
-        </geometry>
       </collision>
       <inertial>
@@ -169,4 +164,12 @@
           <mesh filename="file://$(find robot_model_description)/meshes/dae/Cylinder.003.dae" scale="0.05000 0.05000 0.20000"/>
         </geometry>
+        <surface>
+          <friction>
+            <ode>
+              <mu>1.000000</mu>
+              <mu2>1.000000</mu2>
+            </ode>
+          </friction>
+        </surface>
       </collision>
       <inertial>
@@ -189,4 +192,12 @@
           <mesh filename="file://$(find robot_model_description)/meshes/dae/Cylinder.001.dae" scale="0.05000 0.05000 0.20000"/>
         </geometry>
+        <surface>
+          <friction>
+            <ode>
+              <mu>1.000000</mu>
+              <mu2>1.000000</mu2>
+            </ode>
+          </friction>
+        </surface>
       </collision>
       <inertial>
@@ -209,4 +220,12 @@
           <mesh filename="file://$(find robot_model_description)/meshes/dae/Cylinder.dae" scale="0.05000 0.05000 0.20000"/>
         </geometry>
+        <surface>
+          <friction>
+            <ode>
+              <mu>1.000000</mu>
+              <mu2>1.000000</mu2>
+            </ode>
+          </friction>
+        </surface>
       </collision>
       <inertial>
@@ -223,24 +242,76 @@
       </visual>
     </link>
-    <!--Transmission is important to link the joints ant the controller (see config/rover_controller.yaml)-->
-    <!--
-    <transmission name="${prefix}_wheel_joint_link">
-      <type>transmission_interface/SimpleTransmission</type>
-      <joint name="${prefix}wheel_joint_motor">
+    <!-- Transmission for left back wheel -->
+    <transmission name="wheel_down_left_joint_link">
+    <type>transmission_interface/SimpleTransmission</type>
+    <joint name="wheel_down_left_link_joint">
         <hardwareInterface>hardware_interface/VelocityJointInterface</hardwareInterface>
-      </joint>
-      <actuator name="${prefix}wheel_joint_motor">
+    </joint>
+    <actuator name="left_back_wheel_motor">
         <mechanicalReduction>1</mechanicalReduction>
-      </actuator>
+    </actuator>
     </transmission>
-    <gazebo reference="${prefix}wheel_link">
-      <mu1>5</mu1>
-      <mu2>5</mu2>
-      # <kp>2.75e6</kp>
-      # <kd>8.25e1</kd>
-      # <fdir1>0 0 0</fdir1>
-      # <maxContacts>4</maxContacts>
+    <!-- Transmission for left front wheel -->
+    <transmission name="wheel_up_left_joint_link">
+    <type>transmission_interface/SimpleTransmission</type>
+    <joint name="wheel_up_left_link_joint">
+        <hardwareInterface>hardware_interface/VelocityJointInterface</hardwareInterface>
+    </joint>
+    <actuator name="left_front_wheel_motor">
+        <mechanicalReduction>1</mechanicalReduction>
+    </actuator>
+    </transmission>
+    <!-- Transmission for right back wheel -->
+    <transmission name="wheel_down_right_joint_link">
+    <type>transmission_interface/SimpleTransmission</type>
+    <joint name="wheel_down_right_link_joint">
+        <hardwareInterface>hardware_interface/VelocityJointInterface</hardwareInterface>
+    </joint>
+    <actuator name="right_back_wheel_motor">
+        <mechanicalReduction>1</mechanicalReduction>
+    </actuator>
+    </transmission>
+    <!-- Transmission for right front wheel -->
+    <transmission name="wheel_up_right_joint_link">
+    <type>transmission_interface/SimpleTransmission</type>
+    <joint name="wheel_up_right_link_joint">
+        <hardwareInterface>hardware_interface/VelocityJointInterface</hardwareInterface>
+    </joint>
+    <actuator name="right_front_wheel_motor">
+        <mechanicalReduction>1</mechanicalReduction>
+    </actuator>
+    </transmission>
+    <gazebo reference="wheel_down_left_link">
+    <mu1>5</mu1>
+    <mu2>5</mu2>
+    <!--<kp>2.75e6</kp>
+    <kd>8.25e1</kd>
+    <fdir1>0 0 0</fdir1>
+    <maxContacts>4</maxContacts>-->
     </gazebo>
-    -->
+    <gazebo reference="wheel_up_left_link">
+    <mu1>5</mu1>
+    <mu2>5</mu2>
+    <!--<kp>2.75e6</kp>
+    <kd>8.25e1</kd>
+    <fdir1>0 0 0</fdir1>
+    <maxContacts>4</maxContacts>-->
+    </gazebo>
+    <gazebo reference="wheel_down_right_link">
+    <mu1>5</mu1>
+    <mu2>5</mu2>
+    <!--<kp>2.75e6</kp>
+    <kd>8.25e1</kd>
+    <fdir1>0 0 0</fdir1>
+    <maxContacts>4</maxContacts>-->
+    </gazebo>
+    <gazebo reference="wheel_up_right_link">
+    <mu1>5</mu1>
+    <mu2>5</mu2>
+    <!--<kp>2.75e6</kp>
+    <kd>8.25e1</kd>
+    <fdir1>0 0 0</fdir1>
+    <maxContacts>4</maxContacts>-->
+    </gazebo>
   </xacro:macro>
 </robot>
